File: esp_md3_servo3_sensor3/esp_md3_servo3_sensor3.kicad_pcb (KiCad board)
At the start: 2 copper layers, 75.7 x 69.3 mm, 30 parts, among them J1 Conn_01x02_Pin, U1 ESP32-DEVKITC-32E, U2 LM7805_TO220

Commit message: ミスを修正
Parts:
- moved C1 0.41 mm to (194.2, 113.7)
Other:
- board text added: "Sencor1"
- board text added: "Sencor2"
- board text added: "Sencor3"
Changed lines of the file:
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@@
 		)
 		(fp_text user "${REFERENCE}"
-			(at 2.5 1.85 90)
-			(layer "F.Fab")
+			(at 1.596 -6.714 90)
+			(layer "F.Cu" knockout)
 			(effects
 				(font
-					(size 1 1)
-					(thickness 0.15)
+					(size 1.3 1.3)
+					(thickness 0.2)
 				)
 			)
@@
 			(at 1.25 -3.55 90)
 			(layer "F.SilkS")
+			(hide yes)
 			(effects
 				(font
@@
 			(at 1.25 4.6 90)
 			(layer "F.Fab")
+			(hide yes)
 			(effects
 				(font
@@
 			(layer "F.Fab")
 		)
-		(fp_text user "${REFERENCE}"
-			(at 1.25 2.7 90)
-			(layer "F.Fab")
-			(effects
-				(font
-					(size 1 1)
-					(thickness 0.15)
-				)
-			)
-		)
 		(pad "1" thru_hole roundrect
 			(at 0 0 270)
@@
 			(at 1.25 4.6 90)
 			(layer "F.Fab")
+			(hide yes)
 			(effects
 				(font
@@
 		)
 		(fp_text user "${REFERENCE}"
-			(at 2.5 1.85 90)
-			(layer "F.Fab")
+			(at 3.396 -6.514 90)
+			(layer "F.Cu" knockout)
 			(effects
 				(font
-					(size 1 1)
-					(thickness 0.15)
+					(size 1.3 1.3)
+					(thickness 0.2)
 				)
 			)
@@
 			(at 1.25 4.6 90)
 			(layer "F.Fab")
+			(hide yes)
 			(effects
 				(font
@@
 			(layer "F.Fab")
 		)
-		(fp_text user "${REFERENCE}"
-			(at 1.25 2.7 90)
-			(layer "F.Fab")
-			(effects
-				(font
-					(size 1 1)
-					(thickness 0.15)
-				)
-			)
-		)
 		(pad "1" thru_hole roundrect
 			(at 0 0 270)
@@
 		)
 		(fp_text user "${REFERENCE}"
-			(at 2.5 1.85 90)
-			(layer "F.Fab")
+			(at 2.146 -6.514 90)
+			(layer "F.Cu" knockout)
 			(effects
 				(font
-					(size 1 1)
-					(thickness 0.15)
+					(size 1.3 1.3)
+					(thickness 0.2)
 				)
 			)
@@
 	(footprint "Capacitor_THT:C_Disc_D3.4mm_W2.1mm_P2.50mm"
 		(layer "F.Cu")
-		(at 194.604 113.792)
+		(at 194.2 113.7)
 		(descr "C, Disc series, Radial, pin pitch=2.50mm, , diameter*width=3.4*2.1mm^2, Capacitor, http://www.vishay.com/docs/45233/krseries.pdf")
 		(tags "C Disc series Radial pin pitch 2.50mm  diameter 3.4mm width 2.1mm Capacitor")
@@
 	)
 	(gr_text "3.3V"
-		(at 206.248 131.572 90)
+		(at 204.8 131.3 90)
 		(layer "F.Cu" knockout)
 		(effects
 			(font
-				(size 1.5 1.5)
-				(thickness 0.3)
-				(bold yes)
+				(size 1.3 1.3)
+				(thickness 0.2)
 			)
 			(justify left bottom)
@@
 		)
 	)
+	(gr_text "Sencor3\n"
+		(at 213.9 122.4 90)
+		(layer "F.Cu" knockout)
+		(effects
+			(font
+				(size 1.5 1.5)
+				(thickness 0.3)
+				(bold yes)
+			)
+			(justify left bottom)
+		)
+	)
 	(gr_text "MD2"
 		(at 154.432 114.554 270)
@@
 		)
 	)
+	(gr_text "Sencor2\n"
+		(at 214 132.1 90)
+		(layer "F.Cu" knockout)
+		(effects
+			(font
+				(size 1.5 1.5)
+				(thickness 0.3)
+				(bold yes)
+			)
+			(justify left bottom)
+		)
+	)
 	(gr_text "G"
 		(at 202.946 109.22 90)
@@
 	)
 	(gr_text "3.3V"
-		(at 206.248 121.92 90)
+		(at 204.8 122.4 90)
 		(layer "F.Cu" knockout)
 		(effects
 			(font
-				(size 1.5 1.5)
-				(thickness 0.3)
-				(bold yes)
+				(size 1.3 1.3)
+				(thickness 0.2)
 			)
 			(justify left bottom)
@@
 		)
 	)
-	(gr_text "3.3V"
-		(at 206.248 141.224 90)
+	(gr_text "G"
+		(at 202.946 85.344 90)
 		(layer "F.Cu" knockout)
 		(effects
 			(font
-				(size 1.5 1.5)
-				(thickness 0.3)
+				(size 1 1)
+				(thickness 0.2)
 				(bold yes)
 			)
@@
 		)
 	)
-	(gr_text "G"
-		(at 202.946 85.344 90)
+	(gr_text "3.3V"
+		(at 204.8 141 90)
 		(layer "F.Cu" knockout)
 		(effects
 			(font
-				(size 1 1)
+				(size 1.3 1.3)
 				(thickness 0.2)
+			)
+			(justify left bottom)
+		)
+	)
+	(gr_text "Sencor1"
+		(at 214 142 90)
+		(layer "F.Cu" knockout)
+		(effects
+			(font
+				(size 1.5 1.5)
+				(thickness 0.3)
 				(bold yes)
 			)
@@
 	)
 	(segment
-		(start 191.262 113.792)
-		(end 194.604 113.792)
+		(start 188.722 91.694)
+		(end 186.182 89.154)
 		(width 0.8)
 		(layer "B.Cu")
@@
 	)
 	(segment
-		(start 188.722 91.694)
-		(end 186.182 89.154)
+		(start 191.354 113.7)
+		(end 194.512 113.7)
 		(width 0.8)
 		(layer "B.Cu")
@@
 	)
 	(segment
+		(start 191.135 113.919)
+		(end 191.354 113.7)
+		(width 0.8)
+		(layer "B.Cu")
+		(net 1)
+	)
+	(segment
 		(start 191.516 135.89)
 		(end 194.35 138.724)
@@
 	)
 	(segment
-		(start 164.592 94.295997)
-		(end 163.790997 95.097)
+		(start 194.512 113.7)
+		(end 194.604 113.792)
 		(width 0.8)
 		(layer "B.Cu")
@@
 	)
 	(segment
-		(start 191.135 113.919)
-		(end 191.262 113.792)
+		(start 164.592 94.295997)
+		(end 163.790997 95.097)
 		(width 0.8)
 		(layer "B.Cu")
@@
 	)
 	(segment
-		(start 187.342214 84.936)
+		(start 187.036 84.936)
 		(end 174.244 84.936)
 		(width 0.8)
@@
 	)
 	(segment
-		(start 199.898 97.391786)
-		(end 187.442214 84.936)
+		(start 199.460626 111.360626)
+		(end 194.2 106.1)
 		(width 0.8)
 		(layer "F.Cu")
@@
 	)
 	(segment
-		(start 174.244 84.936)
-		(end 172.52 86.66)
+		(start 199.460626 121.736626)
+		(end 199.460626 111.360626)
 		(width 0.8)
 		(layer "F.Cu")
@@
 	)
 	(segment
-		(start 200.533 122.809)
-		(end 199.898 122.174)
+		(start 172.52 86.66)
+		(end 172.52 95.758)
 		(width 0.8)
 		(layer "F.Cu")
@@
 	)
 	(segment
-		(start 187.442214 84.936)
-		(end 187.342214 84.936)
+		(start 194.2 106.1)
+		(end 194.2 92.1)
 		(width 0.8)
 		(layer "F.Cu")
@@
 	)
 	(segment
-		(start 172.52 86.66)
-		(end 172.52 95.758)
+		(start 194.2 92.1)
+		(end 187.036 84.936)
 		(width 0.8)
 		(layer "F.Cu")
@@
 	)
 	(segment
-		(start 199.898 122.174)
-		(end 199.898 97.391786)
+		(start 200.533 122.809)
+		(end 199.460626 121.736626)
+		(width 0.8)
+		(layer "F.Cu")
+		(net 5)
+	)
+	(segment
+		(start 174.244 84.936)
+		(end 172.52 86.66)
 		(width 0.8)
 		(layer "F.Cu")
@@
 	)
 	(segment
-		(start 198.460625 98.384625)
-		(end 186.182 86.106)
+		(start 195.95 109.85)
+		(end 192.8 106.7)
 		(width 0.8)
 		(layer "F.Cu")
@@
 	)
 	(segment
-		(start 198.460625 110.744)
-		(end 198.460625 98.384625)
+		(start 192.8 92.724)
+		(end 186.182 86.106)
+		(width 0.8)
+		(layer "F.Cu")
+		(net 6)
+	)
+	(segment
+		(start 192.8 106.7)
+		(end 192.8 92.724)
 		(width 0.8)
 		(layer "F.Cu")
@@
 	)
 	(via
-		(at 198.460625 110.744)
+		(at 195.95 109.85)
 		(size 0.6)
 		(drill 0.3)
@@
 	)
 	(segment
-		(start 198.460625 111.592625)
-		(end 203.2 116.332)
+		(start 202.432 116.332)
+		(end 208.422 116.332)
 		(width 0.8)
 		(layer "B.Cu")
@@
 	)
 	(segment
-		(start 208.422 116.332)
-		(end 208.462 116.372)
+		(start 195.95 109.85)
+		(end 202.432 116.332)
 		(width 0.8)
 		(layer "B.Cu")
@@
 	)
 	(segment
-		(start 198.460625 110.744)
-		(end 198.460625 111.592625)
-		(width 0.8)
-		(layer "B.Cu")
-		(net 6)
-	)
-	(segment
-		(start 203.2 116.332)
-		(end 208.422 116.332)
+		(start 208.422 116.332)
+		(end 208.462 116.372)
 		(width 0.8)
 		(layer "B.Cu")
